File: Scanner-zeners.kicad_pcb (KiCad board)
At the start: 2 copper layers, 48 parts, among them J1 Conn_01x04, J2 Battery connector, Q1 BC548, Q2 BC548, Q3 BC548, Q4 BC548, Q5 BC548, Q6 BC548, U1 S4EBL25V, U2 S4EBL25V, U3 PC817, U4 PC817, U5 PC817, U6 4028, U7 S4EBL25V, U8 S4EBL25V

Commit message: Version para back panel lista
Parts:
- removed REF** (x4): MountingHole_3.5mm, Mounting_Holes:MountingHole_3.5mm
- added J3: Battery connector, Connector_PinHeader_2.54mm:PinHeader_1x02_P2.54mm_Vertical, F.Cu at (79.7, 89.2)
- J1: value Conn_01x04 -> Conn_01x20_Male; footprint Pin_Headers:Pin_Header_Straight_1x04_Pitch2.54mm -> Connector_PinHeader_2.54mm:PinHeader_1x20_P2.54mm_Horizontal
- J2: footprint Pin_Headers:Pin_Header_Straight_2x01_Pitch2.54mm -> Connector_PinHeader_2.54mm:PinHeader_1x02_P2.54mm_Vertical
- moved J1 19.9 mm to (50.8, 81.3), turned to 180 degrees
- moved J2 10.6 mm to (84.7, 89.3)
Connections:
- J1 pad 1: /pin0 -> Net-(J1-Pad1)
- J1 pad 2: /pin1 -> Net-(J1-Pad2)
- J1 pad 3: /pin2 -> Net-(J1-Pad3)
- J1 pad 4: /Arduino_GND -> Net-(J1-Pad4)
Routing:
- net /pin0: track 67.3 -> 6.67 mm
- net /pin2: track 56.7 -> 8.52 mm
- net /pin1: track 45.5 -> 16.1 mm
- net /Arduino_GND: track 73.2 -> 49.9 mm
- net +12V: track 273.6 -> 283.3 mm
Other:
- board text added: "M2C relay module M. Senger - INTI 190522"
- board text removed: "M2C relay module M. Senger - INTI - 2018"
